File: Kicad/FlappyBird_Project.kicad_pcb (KiCad board)
At the start: 2 copper layers, 76.2 x 63.5 mm, 15 parts, among them J1 USB_B, Q2 BC846, SW2 SW_MEC_5E, U1 PIC18F4550-IP, U2 M24C02-WMN, Y1 Crystal_GND3

Commit message: Add files via upload
Parts:
- removed SW2: SW_MEC_5E, Button_Switch_SMD:SW_MEC_5GSH9
- added SW1: SW_Omron_B3FS, Button_Switch_SMD:SW_SPST_Omron_B3FS-100xP, F.Cu at (66.0, 88.9)
- J1: footprint Connector_USB:USB_B_OST_USB-B1HSxx_Horizontal -> Connector_USB:USB_B_Amphenol_MUSB-D511_Vertical_Rugged
- moved Q2 5.08 mm to (60.0, 59.5)
- moved D1 5.08 mm to (106.7, 64.4)
- moved G*** 5.08 mm to (119.4, 99.1)
- moved R1 5.08 mm to (106.7, 71.1)
- moved R2 5.08 mm to (72.7, 58.4)
- moved R3 5.08 mm to (57.5, 53.3)
- moved R4 5.08 mm to (55.9, 88.0)
- moved R5 5.08 mm to (71.1, 81.3)
- moved R6 5.08 mm to (71.1, 74.6)
- moved U1 5.08 mm to (81.3, 45.7)
- moved Y1 5.08 mm to (66.0, 68.6)
- moved BZ1 5.08 mm to (63.5, 48.3)
- moved U2 5.08 mm to (60.9, 78.1)
- moved J1 3.57 mm to (113.6, 58.2), turned to 90 degrees
Routing:
- net Net-(J1-D+): track 99.1 -> 86.6 mm
- net Net-(R4-Pad2): track 5.58 -> 8.10 mm
- net GND: track 117.7 -> 119.9 mm
- net Net-(D1-A): track 7.68 -> 9.64 mm
- net Net-(U1-P1A/CCP1/RC2): track 12.6 -> 11.4 mm
