File: Kicad/FlappyBird_Project.kicad_sch (KiCad schematic)
At the start: 14 parts, among them J2 USB_B, Q2 BC846, SW2 SW_MEC_5E, U1 PIC18F4550-IP, U2 M24C02-WMN, Y1 Crystal_GND3

Commit message: Add files via upload
Parts:
- removed J2: USB_B, Connector_USB:USB_B_Lumberg_2411_02_Horizontal, symbol Connector:USB_B
- removed SW2: SW_MEC_5E, Button_Switch_SMD:SW_MEC_5GSH9, symbol Switch:SW_MEC_5E
- added J1: USB_B, Connector_USB:USB_B_Amphenol_MUSB-D511_Vertical_Rugged, symbol Connector:USB_B
- added SW1: SW_Omron_B3FS, Button_Switch_SMD:SW_SPST_Omron_B3FS-100xP, symbol Switch:SW_Omron_B3FS
Connections:
- net GND: now also J1.4 (GND)
- net at D1.2 (A): now also J1.1 (VBUS)
- net at U1.23 (VM/D-/RC4), U1.3 (RA1/AN1): now also J1.2 (D-)
- net at U1.2 (RA0/AN0), U1.24 (VP/D+/RC5): now also J1.3 (D+)
- net at R4.2: now also SW1.1
- net at U1.17 (P1A/CCP1/RC2): now also SW1.2
Changed lines of the file:
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@@
-    )
-  )
-  (symbol (lib_id "power:GND") (at 120.65 124.46 0) (unit 1)
-    (in_bom yes) (on_board yes) (dnp no)
-    (property "Reference" "#PWR09" (at 120.65 130.81 0)
-      (effects (font (size 1.27 1.27)) hide)
-    )
-    (property "Value" "GND" (at 120.65 129.54 0)
-      (effects (font (size 1.27 1.27)))
-    )
-    (property "Footprint" "" (at 120.65 124.46 0)
-      (effects (font (size 1.27 1.27)) hide)
-    )
-    (property "Datasheet" "" (at 120.65 124.46 0)
-      (effects (font (size 1.27 1.27)) hide)
-    )
-    (pin "1")
-    (instances
-      (project "FlappyBird_Project"
-        (path "/b3c59df0-73ae-48d9-8fb2-3e236fac52b9"
-          (reference "#PWR09") (unit 1)
-        )
-      )
     )
   )
   (symbol (lib_id "Connector:USB_B") (at 184.15 46.99 0) (mirror y) (unit 1)
     (in_bom yes) (on_board yes) (dnp no)
-    (property "Reference" "J2" (at 184.15 35.56 0)
+    (property "Reference" "J1" (at 184.15 35.56 0)
       (effects (font (size 1.27 1.27)))
     )
@@
       (effects (font (size 1.27 1.27)))
     )
-    (property "Footprint" "Connector_USB:USB_B_Lumberg_2411_02_Horizontal" (at 180.34 48.26 0)
+    (property "Footprint" "Connector_USB:USB_B_Amphenol_MUSB-D511_Vertical_Rugged" (at 180.34 48.26 0)
       (effects (font (size 1.27 1.27)) hide)
     )
@@
       (project "FlappyBird_Project"
         (path "/b3c59df0-73ae-48d9-8fb2-3e236fac52b9"
-          (reference "J2") (unit 1)
+          (reference "J1") (unit 1)
+        )
+      )
+    )
+  )
+  (symbol (lib_id "power:GND") (at 120.65 124.46 0) (unit 1)
+    (in_bom yes) (on_board yes) (dnp no)
+    (property "Reference" "#PWR09" (at 120.65 130.81 0)
+      (effects (font (size 1.27 1.27)) hide)
+    )
+    (property "Value" "GND" (at 120.65 129.54 0)
+      (effects (font (size 1.27 1.27)))
+    )
+    (property "Footprint" "" (at 120.65 124.46 0)
+      (effects (font (size 1.27 1.27)) hide)
+    )
+    (property "Datasheet" "" (at 120.65 124.46 0)
+      (effects (font (size 1.27 1.27)) hide)
+    )
+    (pin "1")
+    (instances
+      (project "FlappyBird_Project"
+        (path "/b3c59df0-73ae-48d9-8fb2-3e236fac52b9"
+          (reference "#PWR09") (unit 1)
         )
       )
@@
         (path "/b3c59df0-73ae-48d9-8fb2-3e236fac52b9"
           (reference "#PWR07") (unit 1)
-        )
-      )
-    )
-  )
-  (symbol (lib_id "Switch:SW_MEC_5E") (at 152.4 34.29 0) (unit 1)
-    (in_bom yes) (on_board yes) (dnp no) (fields_autoplaced)
-    (property "Reference" "SW2" (at 152.4 25.4 0)
-      (effects (font (size 1.27 1.27)))
-    )
-    (property "Value" "SW_MEC_5E" (at 152.4 27.94 0)
-      (effects (font (size 1.27 1.27)))
-    )
-    (property "Footprint" "Button_Switch_SMD:SW_MEC_5GSH9" (at 152.4 26.67 0)
-      (effects (font (size 1.27 1.27)) hide)
-    )
-    (property "Datasheet" "http://www.apem.com/int/index.php?controller=attachment&id_attachment=1371" (at 152.4 26.67 0)
-      (effects (font (size 1.27 1.27)) hide)
-    )
-    (pin "1")
-    (pin "2")
-    (pin "3")
-    (pin "4")
-    (instances
-      (project "FlappyBird_Project"
-        (path "/b3c59df0-73ae-48d9-8fb2-3e236fac52b9"
-          (reference "SW2") (unit 1)
         )
       )
@@
         )
       )
+    )
+  )
+  (symbol (lib_id "Switch:SW_Omron_B3FS") (at 152.4 34.29 0) (unit 1)
+    (in_bom yes) (on_board yes) (dnp no) (fields_autoplaced)
+    (property "Reference" "SW1" (at 152.4 27.94 0)
+      (effects (font (size 1.27 1.27)))
+    )
+    (property "Value" "SW_Omron_B3FS" (at 152.4 30.48 0)
+      (effects (font (size 1.27 1.27)))
+    )
+    (property "Footprint" "Button_Switch_SMD:SW_SPST_Omron_B3FS-100xP" (at 152.4 29.21 0)
+      (effects (font (size 1.27 1.27)) hide)
+    )
+    (property "Datasheet" "https://omronfs.omron.com/en_US/ecb/products/pdf/en-b3fs.pdf" (at 152.4 29.21 0)
+      (effects (font (size 1.27 1.27)) hide)
+    )
+    (pin "1")
+    (pin "2")
+    (instances
+      (project "FlappyBird_Project"
+        (path "/b3c59df0-73ae-48d9-8fb2-3e236fac52b9"
+          (reference "SW1") (unit 1)
+        )
+      )
